File: Signal-blocker-Minimal/3_RFID Module.kicad_sch (KiCad schematic)
At the start: 3 parts

Commit message: Version 2.1 Update！
Fix some circuit!
More stabler!
Replace all the restrictor and capacitor into 0603 packaging!
create BOM excel,Bill of Material.
Parts:
- removed ?: (no value), ProPrj_Sig-easyedapro:, symbol ProPrj_Sig-easyedapro:Drawing-Symbol_A4
- removed ANTENNA: (no value), ProPrj_Sig-easyedapro:wire, symbol ProPrj_Sig-easyedapro:wire
- removed CK6: 0Ω, ProPrj_Sig-easyedapro:R0603, symbol ProPrj_Sig-easyedapro:0Ω
- added ?: (no value), Signal-blo-easyedapro:, symbol Signal-blo-easyedapro:Drawing-Symbol_A4
- added ANTENNA: (no value), Signal-blo-easyedapro:wire, symbol Signal-blo-easyedapro:wire
- added CK6: 0Ω, Signal-blo-easyedapro:R0603, symbol Signal-blo-easyedapro:0Ω
Connections:
- net GND: now also ANTENNA.1 (GND)
- net RFOUT: now also CK6.1
- new net: ANTENNA.2 (RFOUT), CK6.2
