File: Signal-blocker-Minimal/6_Noise-remove Module.kicad_sch (KiCad schematic)
At the start: 7 parts, among them U9 LM358DR2G

Commit message: Version 2.1 Update！
Fix some circuit!
More stabler!
Replace all the restrictor and capacitor into 0603 packaging!
create BOM excel,Bill of Material.
Parts:
- removed ?: (no value), ProPrj_Sig-easyedapro:, symbol ProPrj_Sig-easyedapro:Drawing-Symbol_A4
- removed C5, C6: 56nF, ProPrj_Sig-easyedapro:C0402, symbol ProPrj_Sig-easyedapro:0402B563K160CT
- removed CK5: 0Ω, ProPrj_Sig-easyedapro:R0603, symbol ProPrj_Sig-easyedapro:0Ω
- removed R4, R5: 100Ω, ProPrj_Sig-easyedapro:R0805, symbol ProPrj_Sig-easyedapro:0805W8F1000T5E
- removed U9: LM358DR2G, ProPrj_Sig-easyedapro:SOIC-8_L5.0-W4.0-P1.27-LS6.0-BL, symbol ProPrj_Sig-easyedapro:LM358DR2G
- added ?: (no value), Signal-blo-easyedapro:, symbol Signal-blo-easyedapro:Drawing-Symbol_A4
- added C5, C6: 56nF, Signal-blo-easyedapro:C0402, symbol Signal-blo-easyedapro:0402B563K160CT
- added CK5: 0Ω, Signal-blo-easyedapro:R0603, symbol Signal-blo-easyedapro:0Ω
- added R4, R5: 100Ω, Signal-blo-easyedapro:R0805, symbol Signal-blo-easyedapro:0805W8F1000T5E
- added U9: LM358DR2G, Signal-blo-easyedapro:SOIC-8_L5.0-W4.0-P1.27-LS6.0-BL, symbol Signal-blo-easyedapro:LM358DR2G
Connections:
- net GND: now also R5.2, U9.4 (GND)
- net RFOUT: now also R4.2, U9.1 (1OUT), U9.2 (1IN-)
- net SIGNAL: now also CK5.2
- net VCC+: now also U9.8 (VCC)
- new net: C5.1, CK5.1
- new net: C5.2, C6.1, R4.1
- new net: C6.2, R5.1, U9.3 (1IN+)
