File: Signal-blocker-Minimal/7_Signal-enhance Module.kicad_sch (KiCad schematic)
At the start: 1 part

Commit message: Version 2.1 Update！
Fix some circuit!
More stabler!
Replace all the restrictor and capacitor into 0603 packaging!
create BOM excel,Bill of Material.
Parts:
- removed ?: (no value), ProPrj_Sig-easyedapro:, symbol ProPrj_Sig-easyedapro:Drawing-Symbol_A4
- added ?: (no value), Signal-blo-easyedapro:, symbol Signal-blo-easyedapro:Drawing-Symbol_A4
Changed lines of the file:
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@@
 	(paper "User" 37.2872 5.6896)
 	(symbol
-		(lib_id "ProPrj_Sig-easyedapro:Drawing-Symbol_A4")
+		(lib_id "Signal-blo-easyedapro:Drawing-Symbol_A4")
 		(at -123.19 13.97 0)
 		(unit 1)
@@
 			)
 		)
-		(property "Footprint" "ProPrj_Sig-easyedapro:"
+		(property "Footprint" "Signal-blo-easyedapro:"
 			(at -123.19 13.97 0)
 			(effects
@@
 		(instances
 			(project ""
-				(path "/d08ab412-bf7b-4d07-89a0-c263cd3ef6f0/68cb6e3d-31a4-4184-8aaf-f8bf86d31cb1"
+				(path "/d6a1a547-a6a2-4474-8af8-e83e8b9a03d8/dcb2c93d-4278-4314-a8aa-3ac89a6c89c3"
 					(reference "?")
 					(unit 1)
